Commit message: update spherization

File: resources/g1_stand/g1_stand_spherized.urdf (robot description, URDF)
Before this commit: robot g1_29dof_with_hand_stand_spherized, 44 links, 43 joints
Links:
- link left_shoulder_yaw_link: geometry collision sphere radius=0.033; collision sphere radius=0.038
- link right_shoulder_yaw_link: geometry collision sphere radius=0.033; collision sphere radius=0.038
- link torso_link: geometry collision sphere radius=0.05; collision sphere radius=0.068

File: resources/g1_up/g1_up_spherized.urdf (robot description, URDF)
Before this commit: robot g1_29dof_with_hand_up_spherized, 46 links, 45 joints
Links:
- link left_shoulder_yaw_link: geometry collision sphere radius=0.033; collision sphere radius=0.038
- link right_shoulder_yaw_link: geometry collision sphere radius=0.033; collision sphere radius=0.038
- link torso_link: geometry collision sphere radius=0.05; collision sphere radius=0.068
